Commit message: Added env var to allow a 7cm forward bumper extension (#92)
* Added env var to allow for extendable front bumper

* Fix weird spacing

* Uploaded bumper extension meshes

* Allowed for different lengths of bumper extensions

File: husky_description/urdf/decorations.urdf.xacro (robot description, xacro)
@@ -23,4 +23,5 @@
 <robot name="husky_decorations" xmlns:xacro="http://ros.org/wiki/xacro">
   <xacro:macro name="husky_decorate">
+    <xacro:property name="husky_bumper_extend" value="$(optenv HUSKY_FORWARD_BUMPER_EXTEND 0)" />
     <!-- Spawn Husky chassis -->
     <link name="top_chassis_link">
@@ -61,8 +62,22 @@
     <!-- Attach front bumper -->
     <joint name="front_bumper" type="fixed">
-      <origin xyz="0.48 0 0.091" rpy="0 0 0" />
+      <origin xyz="${0.48 + husky_bumper_extend / 100.0} 0 0.091" rpy="0 0 0" />
       <parent link="base_link" />
       <child link="front_bumper_link" />
     </joint>
+    <xacro:if value="${husky_bumper_extend}">
+      <link name="front_bumper_extension_link">
+          <visual>
+              <geometry>
+                  <mesh filename="package://husky_description/meshes/bumper_extension.dae" scale="${husky_bumper_extend} 1 1"/>
+              </geometry>
+          </visual>
+      </link>
+      <joint name="front_bumper_extension" type="fixed">
+        <origin xyz="${0.405 + husky_bumper_extend / 200.0} 0 0.091" rpy="0 0 0" />
+        <parent link="base_link" />
+        <child link="front_bumper_extension_link" />
+      </joint>
+    </xacro:if>
     <!-- Spawn rear bumper link -->
     <link name="rear_bumper_link">

File: husky_description/urdf/husky.urdf.xacro (robot description, xacro)
@@ -30,6 +30,12 @@
   <xacro:arg name="kinect_rpy" default="$(optenv HUSKY_KINECT_RPY 0 -0.18 3.14)"/>
   <xacro:arg name="slam_laser_enabled" default="true"/>
+<<<<<<< HEAD
   <xacro:arg name="robot_namespace" default="/"/>
   <!--xacro:arg name="urdf_extras" default="empty.urdf" /-->
+=======
+  <xacro:property name="husky_bumper_extend" value="$(optenv HUSKY_FORWARD_BUMPER_EXTEND 0)" />
+  <xacro:arg name="robot_namespace" default="/" />
+  <xacro:arg name="urdf_extras" default="empty.urdf" />
+>>>>>>> 5f1e46c... Added env var to allow a 7cm forward bumper extension (#92)
   <!-- Included URDF/XACRO Files -->
   <xacro:include filename="$(find husky_description)/urdf/decorations.urdf.xacro"/>
@@ -59,7 +65,11 @@
     </visual>
     <collision>
+<<<<<<< HEAD
       <origin xyz="0 0 ${base_z_size/4}" rpy="0 0 0"/>
+=======
+      <origin xyz="${husky_bumper_extend / 200.0} 0 ${base_z_size/4}" rpy="0 0 0" />
+>>>>>>> 5f1e46c... Added env var to allow a 7cm forward bumper extension (#92)
       <geometry>
-        <box size="${base_x_size} ${base_y_size} ${base_z_size/2}"/>
+        <box size="${base_x_size + husky_bumper_extend / 100.0} ${base_y_size} ${base_z_size/2}"/>
       </geometry>
     </collision>

Commit message: Added some additional frames on the top plates and an environment variable for diabling the user rails

File: husky_description/urdf/decorations.urdf.xacro (robot description, xacro)
@@ -38,18 +38,20 @@
       <child link="top_chassis_link" />
     </joint>
-    <!-- Spawn user rails -->
-    <link name="user_rail_link">
-      <visual>
-        <geometry>
-          <mesh filename="package://husky_description/meshes/user_rail.dae" />
-        </geometry>
-      </visual>
-    </link>
-    <!-- Attach user rails to base link -->
-    <joint name="user_rail" type="fixed">
-      <origin xyz="0.272 0 0.245" rpy="0 0 0" />
-      <parent link="base_link" />
-      <child link="user_rail_link" />
-    </joint>
+    <xacro:if value="$(optenv HUSKY_USER_RAIL_ENABLED true)">
+      <!-- Spawn user rails -->
+      <link name="user_rail_link">
+        <visual>
+          <geometry>
+            <mesh filename="package://husky_description/meshes/user_rail.dae" />
+          </geometry>
+        </visual>
+      </link>
+      <!-- Attach user rails to base link -->
+      <joint name="user_rail" type="fixed">
+        <origin xyz="0.272 0 0.245" rpy="0 0 0" />
+        <parent link="base_link" />
+        <child link="user_rail_link" />
+      </joint>
+    </xacro:if>
     <!-- Spawn front bumper link -->
     <link name="front_bumper_link">
@@ -96,30 +98,86 @@
     <xacro:if value="$(optenv HUSKY_TOP_PLATE_ENABLED true)">
       <!-- Spawn the top plate -->
-      <link name="top_plate_link">
-        <visual>
-          <origin xyz="0 0 0" rpy="0 0 0" />
-          <geometry>
-            <mesh filename="package://husky_description/meshes/top_plate.dae" />
-          </geometry>
-        </visual>
-        <collision>
-          <origin xyz="0 0 0" rpy="0 0 0"/>
-          <geometry>
-            <mesh filename="package://husky_description/meshes/top_plate.dae" />
-          </geometry>
-        </collision>
-        <collision>
-          <!-- Extra collision tag for widgets on top plate -->
-          <geometry>
-            <box size="0.32 0.41 0.09" rpy="0 0 0"/>
-          </geometry>
-        </collision>
-      </link>
-      <!-- Attach top plate -->
-      <joint name="top_plate_joint" type="fixed">
-        <parent link="base_link" />
-        <child link="top_plate_link"/>
-        <origin xyz="0.0812 0 0.245" rpy="0 0 0"/>
-      </joint>
+      <xacro:if value="$(optenv HUSKY_LARGE_TOP_PLATE false)">
+        <link name="top_plate_link">
+          <visual>
+            <origin xyz="0 0 0" rpy="0 0 0" />
+            <geometry>
+              <mesh filename="package://husky_description/meshes/large_top_plate.dae" />
+            </geometry>
+          </visual>
+          <collision>
+            <origin xyz="0 0 0" rpy="0 0 0"/>
+            <geometry>
+              <mesh filename="package://husky_description/meshes/large_top_plate_collision.stl" />
+            </geometry>
+          </collision>
+          <collision>
+            <!-- Extra collision tag for widgets on top plate -->
+            <geometry>
+              <box size="0.32 0.41 0.09" rpy="0 0 0"/>
+            </geometry>
+          </collision>
+        </link>
+        <!-- Attach top plate -->
+        <joint name="top_plate_joint" type="fixed">
+          <parent link="base_link" />
+          <child link="top_plate_link"/>
+          <origin xyz="0.0812 0 0.225" rpy="0 0 0"/>
+        </joint>
+        <!-- Top plate front link -->
+        <joint name="top_plate_front_joint" type="fixed">
+          <parent link="top_plate_link" />
+          <child link="top_plate_front_link"/>
+          <origin xyz="0.4125 0 0.00672" rpy="0 0 0"/>
+        </joint>
+        <!-- Top plate rear link-->
+        <joint name="top_plate_rear_joint" type="fixed">
+          <parent link="top_plate_link" />
+          <child link="top_plate_rear_link"/>
+          <origin xyz="-0.4125 0 0.00672" rpy="0 0 0"/>
+        </joint>
+      </xacro:if>
+      <xacro:unless value="$(optenv HUSKY_LARGE_TOP_PLATE false)">
+        <link name="top_plate_link">
+          <visual>
+            <origin xyz="0 0 0" rpy="0 0 0" />
+            <geometry>
+              <mesh filename="package://husky_description/meshes/top_plate.dae" />
+            </geometry>
+          </visual>
+          <collision>
+            <origin xyz="0 0 0" rpy="0 0 0"/>
+            <geometry>
+              <mesh filename="package://husky_description/meshes/top_plate.dae" />
+            </geometry>
+          </collision>
+          <collision>
+            <!-- Extra collision tag for widgets on top plate -->
+            <geometry>
+              <box size="0.32 0.41 0.09" rpy="0 0 0"/>
+            </geometry>
+          </collision>
+        </link>
+        <!-- Attach top plate -->
+        <joint name="top_plate_joint" type="fixed">
+          <parent link="base_link" />
+          <child link="top_plate_link"/>
+          <origin xyz="0.0812 0 0.245" rpy="0 0 0"/>
+        </joint>
+        <!-- Top plate front link -->
+        <joint name="top_plate_front_joint" type="fixed">
+          <parent link="top_plate_link" />
+          <child link="top_plate_front_link"/>
+          <origin xyz="0.36367 0 0.00639" rpy="0 0 0"/>
+        </joint>
+        <!-- Top plate rear link-->
+        <joint name="top_plate_rear_joint" type="fixed">
+          <parent link="top_plate_link" />
+          <child link="top_plate_rear_link"/>
+          <origin xyz="-0.36633 0 0.00639" rpy="0 0 0"/>
+        </joint>
+      </xacro:unless>
+      <link name="top_plate_front_link"/>
+      <link name="top_plate_rear_link"/>
     </xacro:if>
   </xacro:macro>
