Commit message: husky_Description:Fix my missmerges

File: husky_description/urdf/husky.urdf.xacro (robot description, xacro)
@@ -30,12 +30,7 @@
   <xacro:arg name="kinect_rpy" default="$(optenv HUSKY_KINECT_RPY 0 -0.18 3.14)"/>
   <xacro:arg name="slam_laser_enabled" default="true"/>
-<<<<<<< HEAD
-  <xacro:arg name="robot_namespace" default="/"/>
-  <!--xacro:arg name="urdf_extras" default="empty.urdf" /-->
-=======
   <xacro:property name="husky_bumper_extend" value="$(optenv HUSKY_FORWARD_BUMPER_EXTEND 0)" />
   <xacro:arg name="robot_namespace" default="/" />
   <xacro:arg name="urdf_extras" default="empty.urdf" />
->>>>>>> 5f1e46c... Added env var to allow a 7cm forward bumper extension (#92)
   <!-- Included URDF/XACRO Files -->
   <xacro:include filename="$(find husky_description)/urdf/decorations.urdf.xacro"/>
@@ -65,9 +60,6 @@
     </visual>
     <collision>
-<<<<<<< HEAD
-      <origin xyz="0 0 ${base_z_size/4}" rpy="0 0 0"/>
-=======
+      <!--origin xyz="0 0 ${base_z_size/4}" rpy="0 0 0"/>-->
       <origin xyz="${husky_bumper_extend / 200.0} 0 ${base_z_size/4}" rpy="0 0 0" />
->>>>>>> 5f1e46c... Added env var to allow a 7cm forward bumper extension (#92)
       <geometry>
         <box size="${base_x_size + husky_bumper_extend / 100.0} ${base_y_size} ${base_z_size/2}"/>
